Commit message: fix find package for meshes

File: urdf/meca_500_r3.urdf.xacro (robot description, xacro)
@@ -5,5 +5,5 @@
       <origin xyz="0 0 0" rpy="0 0 0" />
       <geometry>
-        <mesh filename="package://mecademic_description/meshes/meca_500_r3_base.dae" />
+        <mesh filename="package://uclv_aipr_meca500_sim/meshes/meca_500_r3_base.dae" />
       </geometry>
     </visual>
@@ -11,5 +11,5 @@
       <origin xyz="0 0 0" rpy="0 0 0" />
       <geometry>
-        <mesh filename="package://mecademic_description/meshes/meca_500_r3_base_collision.stl" />
+        <mesh filename="package://uclv_aipr_meca500_sim/meshes/meca_500_r3_base_collision.stl" />
       </geometry>
     </collision>
@@ -20,5 +20,5 @@
       <origin xyz="0 0 0" rpy="0 0 0" />
       <geometry>
-        <mesh filename="package://mecademic_description/meshes/meca_500_r3_j1.dae" />
+        <mesh filename="package://uclv_aipr_meca500_sim/meshes/meca_500_r3_j1.dae" />
       </geometry>
     </visual>
@@ -26,5 +26,5 @@
       <origin xyz="0 0 0" rpy="0 0 0" />
       <geometry>
-        <mesh filename="package://mecademic_description/meshes/meca_500_r3_j1_collision.stl" />
+        <mesh filename="package://uclv_aipr_meca500_sim/meshes/meca_500_r3_j1_collision.stl" />
       </geometry>
     </collision>
@@ -42,5 +42,5 @@
       <origin xyz="0 0 0" rpy="0 0 0" />
       <geometry>
-        <mesh filename="package://mecademic_description/meshes/meca_500_r3_j2.dae" />
+        <mesh filename="package://uclv_aipr_meca500_sim/meshes/meca_500_r3_j2.dae" />
       </geometry>
     </visual>
@@ -48,5 +48,5 @@
       <origin xyz="0 0 0" rpy="0 0 0" />
       <geometry>
-        <mesh filename="package://mecademic_description/meshes/meca_500_r3_j2_collision.stl" />
+        <mesh filename="package://uclv_aipr_meca500_sim/meshes/meca_500_r3_j2_collision.stl" />
       </geometry>
     </collision>
@@ -64,5 +64,5 @@
       <origin xyz="0 0 0" rpy="0 0 0" />
       <geometry>
-        <mesh filename="package://mecademic_description/meshes/meca_500_r3_j3.dae" />
+        <mesh filename="package://uclv_aipr_meca500_sim/meshes/meca_500_r3_j3.dae" />
       </geometry>
     </visual>
@@ -70,5 +70,5 @@
       <origin xyz="0 0 0" rpy="0 0 0" />
       <geometry>
-        <mesh filename="package://mecademic_description/meshes/meca_500_r3_j3_collision.stl" />
+        <mesh filename="package://uclv_aipr_meca500_sim/meshes/meca_500_r3_j3_collision.stl" />
       </geometry>
     </collision>
@@ -86,5 +86,5 @@
       <origin xyz="0 0 0" rpy="0 0 0" />
       <geometry>
-        <mesh filename="package://mecademic_description/meshes/meca_500_r3_j4.dae" />
+        <mesh filename="package://uclv_aipr_meca500_sim/meshes/meca_500_r3_j4.dae" />
       </geometry>
     </visual>
@@ -92,5 +92,5 @@
       <origin xyz="0 0 0" rpy="0 0 0" />
       <geometry>
-        <mesh filename="package://mecademic_description/meshes/meca_500_r3_j4_collision.stl" />
+        <mesh filename="package://uclv_aipr_meca500_sim/meshes/meca_500_r3_j4_collision.stl" />
       </geometry>
     </collision>
@@ -108,5 +108,5 @@
       <origin xyz="0 0 0" rpy="0 0 0" />
       <geometry>
-        <mesh filename="package://mecademic_description/meshes/meca_500_r3_j5.dae" />
+        <mesh filename="package://uclv_aipr_meca500_sim/meshes/meca_500_r3_j5.dae" />
       </geometry>
     </visual>
@@ -114,5 +114,5 @@
       <origin xyz="0 0 0" rpy="0 0 0" />
       <geometry>
-        <mesh filename="package://mecademic_description/meshes/meca_500_r3_j5_collision.stl" />
+        <mesh filename="package://uclv_aipr_meca500_sim/meshes/meca_500_r3_j5_collision.stl" />
       </geometry>
     </collision>
@@ -130,5 +130,5 @@
       <origin xyz="0 0 0" rpy="0 0 0" />
       <geometry>
-        <mesh filename="package://mecademic_description/meshes/meca_500_r3_j6.dae" />
+        <mesh filename="package://uclv_aipr_meca500_sim/meshes/meca_500_r3_j6.dae" />
       </geometry>
     </visual>
@@ -136,5 +136,5 @@
       <origin xyz="0 0 0" rpy="0 0 0" />
       <geometry>
-        <mesh filename="package://mecademic_description/meshes/meca_500_r3_j6_collision.stl" />
+        <mesh filename="package://uclv_aipr_meca500_sim/meshes/meca_500_r3_j6_collision.stl" />
       </geometry>
     </collision>
